Commit message: added robo centric architecture plus rainbow robot

File: examples/user_kuka_sinusoid/assets/user_kuka.urdf (robot description, URDF)
Before this commit: robot user_kuka, 9 links, 8 joints
Links:
- added link world
- link base_link: geometry visual cylinder length=0.12 radius=0.09
- link ee_link: geometry visual box size=0.02 0.01 0.06; visual box size=0.02 0.01 0.06
- link link1: geometry visual cylinder length=0.18 radius=0.04
- link link2: geometry visual cylinder length=0.20 radius=0.038
- link link3: geometry visual cylinder length=0.20 radius=0.034
- link link4: geometry visual cylinder length=0.17 radius=0.03
- link link5: geometry visual cylinder length=0.14 radius=0.027
- link link6: geometry visual cylinder length=0.12 radius=0.024
- link link7: geometry visual cylinder length=0.10 radius=0.022
Joints:
- removed joint robot0/joint1
- removed joint robot0/joint2
- removed joint robot0/joint3
- removed joint robot0/joint4
- removed joint robot0/joint5
- removed joint robot0/joint6
- removed joint robot0/joint7
- added joint joint1: type revolute, parent base_link, child link1, origin xyz=0 0 0.06 rpy=0 0 0, axis 0 0 1, limit lower=-2.97 upper=2.97 effort=50.0 velocity=2.0
- added joint joint2: type revolute, parent link1, child link2, origin xyz=0 0 0.18 rpy=0 0 0, axis 0 1 0, limit lower=-2.09 upper=2.09 effort=50.0 velocity=2.0
- added joint joint3: type revolute, parent link2, child link3, origin xyz=0 0 0.20 rpy=0 0 0, axis 0 1 0, limit lower=-2.97 upper=2.97 effort=50.0 velocity=2.0
- added joint joint4: type revolute, parent link3, child link4, origin xyz=0 0 0.20 rpy=0 0 0, axis 1 0 0, limit lower=-2.09 upper=2.09 effort=50.0 velocity=2.0
- added joint joint5: type revolute, parent link4, child link5, origin xyz=0 0 0.17 rpy=0 0 0, axis 0 1 0, limit lower=-2.97 upper=2.97 effort=50.0 velocity=2.0
- added joint joint6: type revolute, parent link5, child link6, origin xyz=0 0 0.14 rpy=0 0 0, axis 1 0 0, limit lower=-2.09 upper=2.09 effort=50.0 velocity=2.0
- added joint joint7: type revolute, parent link6, child link7, origin xyz=0 0 0.12 rpy=0 0 0, axis 0 1 0, limit lower=-3.05 upper=3.05 effort=50.0 velocity=2.0
- added joint world_to_base: type fixed, parent world, child base_link, origin xyz=0 0 0.4 rpy=0 0 0
- joint ee_fixed: origin xyz=0 0 0 rpy=0 0 0 -> xyz=0 0 0.10 rpy=0 0 0

File: examples/user_urdf_asset_override/assets/user_kuka.urdf (robot description, URDF)
Before this commit: robot user_kuka, 9 links, 8 joints
Joints:
- removed joint robot0/joint1
- removed joint robot0/joint2
- removed joint robot0/joint3
- removed joint robot0/joint4
- removed joint robot0/joint5
- removed joint robot0/joint6
- removed joint robot0/joint7
- added joint joint1: type revolute, parent base_link, child link1, origin xyz=0 0 0 rpy=0 0 0, axis 0 0 1, limit lower=-2.97 upper=2.97 effort=50.0 velocity=2.0
- added joint joint2: type revolute, parent link1, child link2, origin xyz=0 0 0 rpy=0 0 0, axis 0 1 0, limit lower=-2.09 upper=2.09 effort=50.0 velocity=2.0
- added joint joint3: type revolute, parent link2, child link3, origin xyz=0 0 0 rpy=0 0 0, axis 0 1 0, limit lower=-2.97 upper=2.97 effort=50.0 velocity=2.0
- added joint joint4: type revolute, parent link3, child link4, origin xyz=0 0 0 rpy=0 0 0, axis 1 0 0, limit lower=-2.09 upper=2.09 effort=50.0 velocity=2.0
- added joint joint5: type revolute, parent link4, child link5, origin xyz=0 0 0 rpy=0 0 0, axis 0 1 0, limit lower=-2.97 upper=2.97 effort=50.0 velocity=2.0
- added joint joint6: type revolute, parent link5, child link6, origin xyz=0 0 0 rpy=0 0 0, axis 1 0 0, limit lower=-2.09 upper=2.09 effort=50.0 velocity=2.0
- added joint joint7: type revolute, parent link6, child link7, origin xyz=0 0 0 rpy=0 0 0, axis 0 1 0, limit lower=-3.05 upper=3.05 effort=50.0 velocity=2.0
