Commit message: fixed SO101 URDF and SLT files

File: robodeploy/description/so101/assets/urdf/so101.urdf (robot description, URDF)
Before this commit: robot so101, 7 links, 6 joints
Links:
- removed link base_link
- removed link gripper_link
- removed link link_fore
- removed link link_shoulder
- removed link link_upper
- removed link link_wrist_pitch
- removed link link_wrist_roll
- added link base, mass 0.147; collision mesh filename=assets/base_motor_holder_so101_v1.stl; collision mesh filename=assets/base_so101_v2.stl
- added link baseframe, mass 1e-9
- added link gripper, mass 0.087; collision mesh filename=assets/sts3215_03a_v1.stl; collision mesh filename=assets/wrist_roll_follower_so101_v1.stl
- added link gripperframe, mass 1e-9
- added link lower_arm, mass 0.104; collision mesh filename=assets/motor_holder_so101_wrist_v1.stl; collision mesh filename=assets/sts3215_03a_v1.stl
- added link moving_jaw_so101_v1, mass 0.012; collision mesh filename=assets/moving_jaw_so101_v1.stl; visual mesh filename=assets/moving_jaw_so101_v1.stl
- added link shoulder, mass 0.100006; collision mesh filename=assets/motor_holder_so101_base_v1.stl; collision mesh filename=assets/rotation_pitch_so101_v1.stl
- added link upper_arm, mass 0.103; collision mesh filename=assets/sts3215_03a_v1.stl; collision mesh filename=assets/upper_arm_so101_v1.stl
- added link wrist, mass 0.079; collision mesh filename=assets/sts3215_03a_no_horn_v1.stl; collision mesh filename=assets/wrist_roll_pitch_so101_v2.stl
Joints:
- removed joint elbow_flex
- removed joint gripper
- removed joint shoulder_lift
- removed joint shoulder_pan
- removed joint wrist_flex
- removed joint wrist_roll
- added joint 1: type revolute, parent base, child shoulder, origin xyz=-0.124202 -0.168068 0.0948817 rpy=3.14159 4.18253e-17 -3.14159, axis 0 0 1, limit lower=-1.91986 upper=1.91986 effort=10 velocity=10
- added joint 2: type revolute, parent shoulder, child upper_arm, origin xyz=-0.0303992 -0.0182778 -0.0542 rpy=-1.5708 -1.5708 0, axis 0 0 1, limit lower=-1.74533 upper=1.74533 effort=10 velocity=10
- added joint 3: type revolute, parent upper_arm, child lower_arm, origin xyz=-0.11257 -0.028 2.09886e-16 rpy=-3.63608e-16 8.74301e-16 1.5708, axis 0 0 1, limit lower=-1.74533 upper=1.5708 effort=10 velocity=10
- added joint 4: type revolute, parent lower_arm, child wrist, origin xyz=-0.1349 0.0052 8.44651e-17 rpy=4.02456e-15 8.67362e-16 -1.5708, axis 0 0 1, limit lower=-1.65806 upper=1.65806 effort=10 velocity=10
- added joint 5: type revolute, parent wrist, child gripper, origin xyz=2.77556e-16 -0.0611 0.0181 rpy=1.5708 0.0486795 3.14159, axis 0 0 1, limit lower=-2.74385 upper=2.84121 effort=10 velocity=10
- added joint 6: type revolute, parent gripper, child moving_jaw_so101_v1, origin xyz=0.0202 0.0188 -0.0234 rpy=1.5708 -5.24284e-08 -1.41553e-15, axis 0 0 1, limit lower=-0.174533 upper=1.74533 effort=10 velocity=10
- added joint baseframe_frame: type fixed, parent base, child baseframe, origin xyz=-0.163038 -0.168068 0.0324817 rpy=1.6144e-15 7.84513e-18 1.33799e-15, axis 0 0 0
- added joint gripperframe_frame: type fixed, parent gripper, child gripperframe, origin xyz=-0.0079 -0.000218121 -0.0981274 rpy=-0 1.5708 0, axis 0 0 0
